File: SG3525 Solar Inverter/H Bridge/kicad/kicad.kicad_pcb (KiCad board)
At the start: 2 copper layers, 72 parts, among them J1 Conn_01x02_Pin, Q1 IRF740, Q2 IRF740, Q3 S8050, Q4 S8050, Q5 IRF740, Q6 IRF740, U1 SG3525, U2 PC817, U3 LM358, U4 PC817

Commit message: WORKING ON H Bridge kicad
Parts:
- removed the C1 at (143.7, 97.4)
- added C4: 100nF, Capacitor_THT:C_Disc_D7.0mm_W2.5mm_P5.00mm, F.Cu at (128.7, 141.0)
- added C9: 10uF 25V, Capacitor_THT:C_Radial_D5.0mm_H11.0mm_P2.00mm, F.Cu at (141.2, 128.6)
- added R34: 370, Resistor_THT:R_Axial_DIN0207_L6.3mm_D2.5mm_P7.62mm_Horizontal, F.Cu at (133.5, 141.2)
- added R35: 20k, Resistor_THT:R_Axial_DIN0207_L6.3mm_D2.5mm_P7.62mm_Horizontal, F.Cu at (123.5, 141.2)
- added RV5: 150k, Potentiometer_THT:Potentiometer_Bourns_3296W_Vertical, F.Cu at (116.6, 139.8)
- moved D1 257.8 mm to (-134.5, 110.9)
- moved D10 257.8 mm to (-73.1, 66.3)
- moved D4 257.8 mm to (-147.3, 81.2)
- moved D5 257.8 mm to (-147.3, 84.5)
- moved D7 257.8 mm to (-148.6, 60.6)
- moved D9 257.8 mm to (-72.5, 78.5)
- moved RV1 257.8 mm to (-124.8, 109.7)
- moved C8 257.8 mm to (-88.9, 146.0)
- moved D2 257.8 mm to (-104.4, 130.5)
- moved D6 257.8 mm to (-139.5, 79.2)
- moved D8 257.8 mm to (-64.2, 76.5)
- moved J1 257.8 mm to (-135.8, 92.1)
- moved R1 257.8 mm to (-135.7, 98.3)
- moved R10 257.8 mm to (-84.1, 70.2)
- moved R11 257.8 mm to (-84.1, 74.3)
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Connections:
- Q4 pad 3: /pc1 -> /pc2
- R27 pad 2: /pc1 -> /pc2
- R29 pad 1: /pc1 -> /pc2
- R31 pad 1: /pc1 -> /pc2
- U4 pad 3: /pc1 -> /pc2
Other:
- board outline added: 92.9 x 61.7 mm

Commit message: WORKING ON H Bridge kicad
Parts:
- moved R8 347.9 mm to (184.1, 138.0), turned to -90 degrees
- moved R4 329.3 mm to (162.2, 138.1), turned to -90 degrees
- moved D5 328.5 mm to (177.0, 137.3)
- moved D6 321.7 mm to (175.7, 143.4)
- moved RV3 319.4 mm to (168.8, 144.3), turned to -90 degrees
- moved R6 315.8 mm to (152.9, 121.6), turned to 180 degrees
- moved R7 308.4 mm to (145.2, 127.1)
- moved R5 302.0 mm to (136.2, 133.2)
- moved D7 272.9 mm to (114.6, 132.8)
- moved R10 268.2 mm to (178.8, 123.1), turned to 180 degrees
- moved R11 260.8 mm to (171.1, 127.9)
- moved R13 255.6 mm to (166.5, 132.7)
- moved R9 251.9 mm to (157.3, 138.1), turned to -90 degrees
- moved D10 231.5 mm to (148.7, 132.9)
- moved RV4 229.9 mm to (151.2, 144.3), turned to -90 degrees
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Other:
- board size 92.9 x 61.7 mm -> 92.9 x 65.5 mm
