File: SG3525 Solar Inverter/H Bridge/kicad/kicad.kicad_pcb (KiCad board)
At the start: 2 copper layers, 106.7 x 65.5 mm, 79 parts, among them J2 Screw_Terminal_01x02, J3 Screw_Terminal_01x02, J4 Screw_Terminal_01x02, Q1 IRF740, Q2 IRF740, Q3 S8050, Q4 S8050, Q5 IRF740, Q6 IRF740, U1 SG3525, U2 PC817, U3 LM358, U4 PC817

Commit message: WORKING ON H Bridge kicad
Parts:
- added C11: 0.1uF 400V, Capacitor_THT:C_Rect_L13.5mm_W5.0mm_P10.00mm_FKS3_FKP3_MKS4, F.Cu at (154.2, 84.9)
- added J1: Screw_Terminal_01x01, Connector_Wire:SolderWire-0.127sqmm_1x01_D0.48mm_OD1mm, F.Cu at (137.9, 80.2)
- added J5: Screw_Terminal_01x01, Connector_Wire:SolderWire-0.127sqmm_1x01_D0.48mm_OD1mm, F.Cu at (153.2, 80.0)
- added Q7: BC547, Package_TO_SOT_THT:TO-92_Inline, F.Cu at (122.9, 103.3)
- added R19: 390k, Resistor_THT:R_Axial_DIN0207_L6.3mm_D2.5mm_P7.62mm_Horizontal, F.Cu at (163.8, 109.2)
- added R36: 10k, Resistor_THT:R_Axial_DIN0207_L6.3mm_D2.5mm_P7.62mm_Horizontal, F.Cu at (126.8, 110.0)
- added R37: 100k, Resistor_THT:R_Axial_DIN0207_L6.3mm_D2.5mm_P7.62mm_Horizontal, F.Cu at (126.7, 114.8)
- added R38: 47R, Resistor_THT:R_Axial_Power_L25.0mm_W6.4mm_P30.48mm, F.Cu at (118.4, 85.7)
- R30: value 0 -> 390k
- moved R30 31.2 mm to (178.2, 119.3), turned to 180 degrees
- moved Q1 12.4 mm to (112.1, 76.9)
- moved Q2 11.7 mm to (127.4, 76.9)
- moved Q5 11.2 mm to (142.8, 76.9)
- moved Q6 11.2 mm to (158.1, 76.9)
- moved C7 9.52 mm to (185.8, 101.7)
- moved C2 9.02 mm to (171.6, 87.7)
- moved D11 9.02 mm to (177.6, 92.6)
- moved D12 9.02 mm to (188.0, 77.2)
- moved D13 9.02 mm to (177.6, 87.0)
- moved D14 9.02 mm to (188.0, 81.9)
- moved R27 7.13 mm to (170.9, 109.8)
- moved R28 7.13 mm to (170.9, 114.4)
- moved D3 7.06 mm to (115.0, 101.1)
- moved R16 7.06 mm to (101.5, 108.6)
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Connections:
- D10 pad 1: /SD -> /TR1
- D10 pad 2: /HV_LED -> Net-(D10-A)
- D7 pad 1: /SD -> /TR1
- D7 pad 2: /LV_LED -> Net-(D7-A)
- R13 pad 1: /HV_LED -> Net-(D10-A)
- R13 pad 2: Net-(R13-Pad2) -> /HV_LED
- R30 pad 1: Net-(C6-Pad2) -> GND
- R30 pad 2: /Neutral -> /LV_LED
- R5 pad 1: /LV_LED -> Net-(D7-A)
- R5 pad 2: Net-(R5-Pad2) -> /LV_LED
- U3 pad 1: Net-(R5-Pad2) -> /LV_LED
- U3 pad 7: Net-(R13-Pad2) -> /HV_LED
Routing:
- net GND: track 317.0 -> 0.00 mm
- net GND2: track 168.0 -> 0.00 mm
- net /Live: track 150.5 -> 0.00 mm
- net +12V: track 125.0 -> 0.00 mm
- net +325V: track 101.5 -> 0.00 mm
- net /INV: track 92.1 -> 0.00 mm
- net /5V VREF: track 86.8 -> 0.00 mm, vias 3 -> 0
- net /LV_LED: track 63.9 -> 0.00 mm
- net /OUTB: track 50.6 -> 0.00 mm
- net /SD: track 49.1 -> 0.00 mm
- net /LMB: track 38.9 -> 0.00 mm
- net /HV_LED: track 31.2 -> 0.00 mm
- net /OUTA: track 30.5 -> 0.00 mm
- net /COMP: track 26.4 -> 0.00 mm
- net /LMA: track 23.8 -> 0.00 mm, vias 1 -> 0
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Other:
- board size 106.7 x 65.5 mm -> 106.7 x 75.3 mm

Commit message: WORKING ON H Bridge kicad
Parts:
- added H4: MountingHole, MountingHole:MountingHole_3.2mm_M3_Pad_Via, F.Cu at (171.9, 95.8)
- added J6: Conn_01x02_Socket, Connector_PinHeader_2.54mm:PinHeader_1x02_P2.54mm_Vertical, F.Cu at (184.3, 78.0)
- C7: footprint Capacitor_THT:C_Radial_D10.0mm_H12.5mm_P5.00mm -> Capacitor_THT:C_Radial_D5.0mm_H11.0mm_P2.00mm
- D15, D4, D5, D8: footprint Diode_SMD:D_MiniMELF -> Diode_THT:D_DO-35_SOD27_P7.62mm_Horizontal
- moved D5 8.07 mm to (174.7, 145.0), turned to 90 degrees
- moved D15 6.56 mm to (182.5, 119.4)
- moved D4 6.41 mm to (114.3, 146.2)
- moved D13 5.85 mm to (177.8, 92.9)
- moved D14 5.85 mm to (188.3, 87.8)
- moved D12 5.85 mm to (188.2, 83.1)
- moved D11 5.85 mm to (177.8, 98.5)
- moved C3 4.80 mm to (105.3, 132.8)
- moved C7 3.59 mm to (184.9, 105.2)
- moved D6 3.26 mm to (178.9, 142.7)
- moved D7 3.15 mm to (111.4, 132.9)
- moved R8 2.78 mm to (186.9, 138.2)
- moved C4 2.61 mm to (131.1, 132.8), turned to 180 degrees
- moved C9 2.19 mm to (140.0, 124.8)
- moved D8 2.16 mm to (143.4, 135.4)
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Connections:
- D11 pad 2: /Live -> /L_VFB
- D12 pad 1: /Live -> /L_VFB
- D13 pad 2: GND2 -> /N_VFB
- D14 pad 1: GND2 -> /N_VFB
Other:
- board text added: "2026/10"
- board text added: "FB"
- board text added: "L"
- board text added: "N"
- board text added: "TIVANA INVERTER V1"
- board text added: "TIVANA LOW/HIGH FREQUENCY INVERTER V1"
