File: SG3525 Solar Inverter/H Bridge/kicad/kicad.kicad_pcb (KiCad board)
At the start: 2 copper layers, 106.7 x 75.3 mm, 89 parts, among them J1 Screw_Terminal_01x01, J2 Screw_Terminal_01x02, J3 Screw_Terminal_01x02, J4 Screw_Terminal_01x02, J5 Screw_Terminal_01x01, J6 Conn_01x02_Socket, Q1 IRF740, Q2 IRF740, Q3 S8050, Q4 S8050, Q5 IRF740, Q6 IRF740, Q7 BC547, U1 SG3525, U2 PC817, U3 LM358, U4 PC817

Commit message: WORKING ON H Bridge kicad
Parts:
- moved C1 79.4 mm to (49.5, 33.2)
- moved C2 79.4 mm to (110.4, 37.1)
- moved C3 79.4 mm to (44.1, 82.2)
- moved C4 79.4 mm to (69.8, 82.2)
- moved C5 79.4 mm to (68.3, 54.5)
- moved C6 79.4 mm to (102.9, 52.9)
- moved C7 79.4 mm to (123.7, 54.6)
- moved C8 79.4 mm to (38.1, 73.1)
- moved C9 79.4 mm to (78.7, 74.2)
- moved D11 79.4 mm to (116.5, 47.9)
- moved D12 79.4 mm to (127.0, 32.5)
- moved D13 79.4 mm to (116.6, 42.3)
- moved D14 79.4 mm to (127.0, 37.2)
- moved D15 79.4 mm to (121.2, 68.8)
- moved D3 79.4 mm to (53.7, 50.5)
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
Commit message: WORKING ON H Bridge kicad
Parts:
- added C12: 2.2uF, Capacitor_THT:C_Disc_D7.0mm_W2.5mm_P5.00mm, F.Cu at (113.6, 133.1)
- added C13: 100uF, Capacitor_THT:C_Disc_D7.0mm_W2.5mm_P5.00mm, F.Cu at (113.6, 137.2)
- added J10: Conn_01x02_Socket, Connector_PinHeader_2.54mm:PinHeader_1x02_P2.54mm_Vertical, F.Cu at (117.1, 113.2)
- added J7: Conn_01x02_Socket, Connector_PinHeader_2.54mm:PinHeader_1x02_P2.54mm_Vertical, F.Cu at (103.3, 113.2)
- added J8: Conn_01x02_Socket, Connector_PinHeader_2.54mm:PinHeader_1x02_P2.54mm_Vertical, F.Cu at (107.9, 113.2)
- added J9: Conn_01x02_Socket, Connector_PinHeader_2.54mm:PinHeader_1x02_P2.54mm_Vertical, F.Cu at (112.5, 113.2)
- added R39: 33k, Resistor_THT:R_Axial_DIN0207_L6.3mm_D2.5mm_P7.62mm_Horizontal, F.Cu at (102.6, 120.1)
- added R40: 10M, Resistor_THT:R_Axial_DIN0207_L6.3mm_D2.5mm_P7.62mm_Horizontal, F.Cu at (102.6, 124.1)
- added R41: 33k, Resistor_THT:R_Axial_DIN0207_L6.3mm_D2.5mm_P7.62mm_Horizontal, F.Cu at (102.6, 128.2)
- added R42: 33k, Resistor_THT:R_Axial_DIN0207_L6.3mm_D2.5mm_P7.62mm_Horizontal, F.Cu at (102.6, 132.2)
- added RV6: 10k, Potentiometer_THT:Potentiometer_Bourns_3296W_Vertical, F.Cu at (119.9, 121.2)
- added U5: PC817, Package_DIP:DIP-4_W7.62mm, F.Cu at (113.4, 126.5)
- C7: value 470uF 400V -> 10uF 400V
Connections:
- C7 pad 2: GND -> Net-(D12-A)
- D15 pad 2: GND -> Net-(D15-A)
- R14 pad 1: /INV -> Net-(R14-Pad1)
- R14 pad 2: Net-(D11-K) -> /INV
- R15 pad 1: GND -> Net-(D15-A)
