File: SG3525 Solar Inverter/H Bridge/kicad/kicad.kicad_sch (KiCad schematic)
At the start: 69 parts, among them J1 Conn_01x02_Pin, Q1 IRF740, Q2 IRF740, Q3 S8050, Q4 S8050, Q5 IRF740, Q6 IRF740, U1 SG3525, U2 PC817, U3 LM358, U4 PC817

Commit message: WORKING ON H Bridge kicad
Parts:
- added C4: 100nF, Capacitor_THT:C_Disc_D7.0mm_W2.5mm_P5.00mm, symbol Device:C_Small
- added C9: 10uF 25V, Capacitor_THT:C_Radial_D5.0mm_H11.0mm_P2.00mm, symbol Device:C_Polarized_Small
- added R34: 370, Resistor_THT:R_Axial_DIN0207_L6.3mm_D2.5mm_P7.62mm_Horizontal, symbol Device:R
- added R35: 20k, Resistor_THT:R_Axial_DIN0207_L6.3mm_D2.5mm_P7.62mm_Horizontal, symbol Device:R
- added RV5: 150k, Potentiometer_THT:Potentiometer_Bourns_3296W_Vertical, symbol Device:R_Potentiometer
Connections:
- net CT: now also C4.2, R34.1
- net DISCH: now also R34.2
- net GND: now also C4.1, C9.2, RV5.2, RV5.3
- net RT: now also R35.2
- net SS: now also C9.1
- net pc1: no longer Q4.3 (C), R27.2, R29.1, R31.1, U4.3
- new net: R35.1, RV5.1
- new net pc2: Q4.3 (C), R27.2, R29.1, R31.1, U4.3
Other:
- moved on the sheet: C1

Commit message: WORKING ON H Bridge kicad
Changed lines of the file:
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@@
 		(in_pos_files yes)
 		(dnp no)
-		(fields_autoplaced yes)
 		(property "Reference" "R14"
 			(at 218.44 139.6999 0)
@@
 		)
 		(property "Value" "33k"
-			(at 218.44 142.2399 0)
+			(at 215.9 143.002 90)
 			(show_name no)
 			(do_not_autoplace no)
@@
 		(in_pos_files yes)
 		(dnp no)
-		(fields_autoplaced yes)
 		(property "Reference" "R15"
 			(at 218.44 153.6699 0)
@@
 		)
 		(property "Value" "10k"
-			(at 218.44 156.2099 0)
-			(show_name no)
-			(do_not_autoplace no)
+			(at 215.9 156.972 90)
+			(show_name no)
+			(do_not_autoplace no)
