File: SG3525 Solar Inverter/H Bridge/kicad/kicad.kicad_sch (KiCad schematic)
At the start: 75 parts, among them J2 Screw_Terminal_01x02, J3 Screw_Terminal_01x02, J4 Screw_Terminal_01x02, Q1 IRF740, Q2 IRF740, Q3 S8050, Q4 S8050, Q5 IRF740, Q6 IRF740, U1 SG3525, U2 PC817, U3 LM358, U4 PC817

Commit message: WORKING ON H Bridge kicad
Parts:
- added H1, H2, H3: MountingHole, MountingHole:MountingHole_3.2mm_M3_Pad_Via, symbol Mechanical:MountingHole
- C10: value 1000uF 25V -> 1000uF 325V
- C3: value 100nF -> 2.2uF
Connections:
- net GND: no longer J3.2 (Pin_2), Q2.3 (S), Q6.3 (S), R21.2, R33.2
- net pc1: no longer Q3.3 (C), R20.1, R24.2
- net pc2: no longer Q4.3 (C), R27.2, R31.1
- net Neutral renamed GND2
- net GND2: now also J3.2 (Pin_2), Q2.3 (S), Q6.3 (S), R21.2, R33.2
- new net: Q4.3 (C), R27.2, R31.1
- new net: Q3.3 (C), R20.1, R24.2

Commit message: WORKING ON H Bridge kicad
Parts:
- added C11: 0.1uF 400V, Capacitor_THT:C_Rect_L13.5mm_W5.0mm_P10.00mm_FKS3_FKP3_MKS4, symbol Device:C
- added Q7: BC547, Package_TO_SOT_THT:TO-92_Inline, symbol Transistor_BJT:BC547
- added R19, R30: 390k, Resistor_THT:R_Axial_DIN0207_L6.3mm_D2.5mm_P7.62mm_Horizontal, symbol Device:R
- added R36, R38: 10k, Resistor_THT:R_Axial_DIN0207_L6.3mm_D2.5mm_P7.62mm_Horizontal, symbol Device:R
- added R37: 100k, Resistor_THT:R_Axial_DIN0207_L6.3mm_D2.5mm_P7.62mm_Horizontal, symbol Device:R
Connections:
- net GND: now also Q7.3 (E), R19.1, R30.1, R37.1
- net GND2: now also R38.1
- net HV_LED: now also R13.2, U3.7, R19.2; no longer D10.2 (A), R13.1
- net LV_LED: now also R5.2, U3.1, R30.2; no longer D7.2 (A), R5.1
- net Live: now also C11.2
- net SD: now also Q7.1 (C); no longer D10.1 (K), D7.1 (K)
- new net: D10.2 (A), R13.1
- new net: Q7.2 (B), R36.1
- new net: D7.2 (A), R5.1
- new net: C11.1, R38.2
- new net TR1: D10.1 (K), D7.1 (K), R36.2, R37.2
Other:
- note added: "SNUBBER CIRCUIT"
- moved on the sheet: C1, C2, C3, C4, C5, C6, C9, D1, D10, D16, D3, D5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

Commit message: WORKING ON H Bridge kicad
Parts:
- R38: value 10k -> 47R; footprint Resistor_THT:R_Axial_DIN0207_L6.3mm_D2.5mm_P7.62mm_Horizontal -> Resistor_THT:R_Axial_Power_L25.0mm_W6.4mm_P30.48mm
Other:
- title: SG3525 H Bridge -> SG3525 Full Bridge Inverter
Changed lines of the file:
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@@
 	(paper "A4")
 	(title_block
-		(title "SG3525 H Bridge")
+		(title "SG3525 Full Bridge Inverter")
 		(date "2026-09-27")
 		(rev "0")
@@
 			)
 		)
-		(property "Value" "10k"
+		(property "Value" "47R"
 			(at 257.81 65.024 90)
 			(show_name no)
@@
 			)
 		)
-		(property "Footprint" "Resistor_THT:R_Axial_DIN0207_L6.3mm_D2.5mm_P7.62mm_Horizontal"
+		(property "Footprint" "Resistor_THT:R_Axial_Power_L25.0mm_W6.4mm_P30.48mm"
 			(at 259.588 64.77 90)
 			(hide yes)

Commit message: WORKING ON H Bridge kicad
Parts:
- added J1, J5: Screw_Terminal_01x01, Connector_Wire:SolderWire-0.127sqmm_1x01_D0.48mm_OD1mm, symbol Connector:Screw_Terminal_01x01
Connections:
- net GND2: now also J5.1 (Pin_1)
- net Live: now also J1.1 (Pin_1)
Changed lines of the file:
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@@
 		(company "Tivana")
 	)
+	(rectangle
+		(start 191.77 127)
+		(end 270.51 165.1)
+		(stroke
+			(width 1)
+			(type solid)
+			(color 255 35 19 1)
+		)
+		(fill
+			(type none)
+		)
+	)
 	(text "HV ALARMS"
 		(exclude_from_sim no)
@@
 	(wire
 		(pts
+			(xy 264.16 58.42) (xy 273.05 58.42)
+		)
+		(stroke
+			(width 0)
+			(type default)
+		)
+	)
+	(wire
+		(pts
 			(xy 240.03 40.64) (xy 245.11 40.64)
 		)
@@
 	(wire
 		(pts
+			(xy 264.16 62.23) (xy 273.05 62.23)
+		)
+		(stroke
+			(width 0)
+			(type default)
+		)
+	)
+	(wire
+		(pts
 			(xy 17.78 49.53) (xy 22.86 49.53)
 		)
@@
 		)
 	)
+	(label "Neutral"
+		(at 269.24 62.23 180)
+		(effects
+			(font
+				(size 1.27 1.27)
+			)
+			(justify right bottom)
+		)
+	)
 	(label "TR1"
 		(at 152.4 128.27 0)
@@
 	)
 	(label "Live"
+		(at 269.24 58.42 180)
+		(effects
+			(font
+				(size 1.27 1.27)
+			)
+			(justify right bottom)
+		)
+	)
+	(label "Live"
 		(at 16.51 104.14 0)
 		(effects
@@
 	)
 	(symbol
+		(lib_id "Connector:Screw_Terminal_01x01")
+		(at 278.13 58.42 0)
+		(unit 1)
+		(body_style 1)
+		(exclude_from_sim no)
+		(in_bom yes)
+		(on_board yes)
+		(in_pos_files yes)
+		(dnp no)
+		(fields_autoplaced yes)
+		(property "Reference" "J1"
+			(at 280.67 58.4199 0)
+			(show_name no)
+			(do_not_autoplace no)
+			(effects
+				(font
+					(size 1.27 1.27)
+				)
+				(justify left)
+			)
+		)
+		(property "Value" "Screw_Terminal_01x01"
+			(at 280.67 59.6899 0)
+			(hide yes)
+			(show_name no)
+			(do_not_autoplace no)
+			(effects
+				(font
+					(size 1.27 1.27)
+				)
+				(justify left)
+			)
+		)
+		(property "Footprint" "Connector_Wire:SolderWire-0.127sqmm_1x01_D0.48mm_OD1mm"
+			(at 278.13 58.42 0)
+			(hide yes)
+			(show_name no)
+			(do_not_autoplace no)
+			(effects
+				(font
+					(size 1.27 1.27)
+				)
+			)
+		)
+		(property "Datasheet" ""
+			(at 278.13 58.42 0)
+			(hide yes)
+			(show_name no)
+			(do_not_autoplace no)
+			(effects
+				(font
+					(size 1.27 1.27)
+				)
+			)
+		)
+		(property "Description" "Generic screw terminal, single row, 01x01, script generated (kicad-library-utils/schlib/autogen/connector/)"
+			(at 278.13 58.42 0)
+			(hide yes)
+			(show_name no)
+			(do_not_autoplace no)
+			(effects
+				(font
+					(size 1.27 1.27)
+				)
+			)
+		)
+		(pin "1"
+		)
+		(instances
+			(project "kicad"
+				(path "/40e0f264-5d7d-4080-96f9-03b6d8dad596"
+					(reference "J1")
+					(unit 1)
+				)
+			)
+		)
+	)
+	(symbol
 		(lib_id "power:GND")
 		(at 175.26 123.19 0)
@@
 					(unit 1)
 				)
+			)
+		)
+	)
+	(symbol
+		(lib_id "Connector:Screw_Terminal_01x01")
+		(at 278.13 62.23 0)
+		(unit 1)
+		(body_style 1)
+		(exclude_from_sim no)
+		(in_bom yes)
+		(on_board yes)
+		(in_pos_files yes)
+		(dnp no)
+		(fields_autoplaced yes)
+		(property "Reference" "J5"
+			(at 280.67 62.2299 0)
+			(show_name no)
+			(do_not_autoplace no)
+			(effects
+				(font
+					(size 1.27 1.27)
+				)
+				(justify left)
+			)
+		)
+		(property "Value" "Screw_Terminal_01x01"
+			(at 280.67 63.4999 0)
+			(hide yes)
+			(show_name no)
+			(do_not_autoplace no)
+			(effects
+				(font
+					(size 1.27 1.27)
+				)
+				(justify left)
+			)
+		)
+		(property "Footprint" "Connector_Wire:SolderWire-0.127sqmm_1x01_D0.48mm_OD1mm"
+			(at 278.13 62.23 0)
+			(hide yes)
+			(show_name no)
+			(do_not_autoplace no)
+			(effects
+				(font
+					(size 1.27 1.27)
+				)
+			)
+		)
+		(property "Datasheet" ""
+			(at 278.13 62.23 0)
+			(hide yes)
+			(show_name no)
+			(do_not_autoplace no)
+			(effects
+				(font
+					(size 1.27 1.27)
+				)
+			)
+		)
+		(property "Description" "Generic screw terminal, single row, 01x01, script generated (kicad-library-utils/schlib/autogen/connector/)"
+			(at 278.13 62.23 0)
+			(hide yes)
+			(show_name no)
+			(do_not_autoplace no)
+			(effects
+				(font
+					(size 1.27 1.27)
+				)
+			)
+		)
+		(pin "1"
+		)
+		(instances
+			(project "kicad"
+				(path "/40e0f264-5d7d-4080-96f9-03b6d8dad596"
+					(reference "J5")
+					(unit 1)
+				)

Commit message: WORKING ON H Bridge kicad
Parts:
- added H4: MountingHole, MountingHole:MountingHole_3.2mm_M3_Pad_Via, symbol Mechanical:MountingHole
- added J6: Conn_01x02_Socket, Connector_PinHeader_2.54mm:PinHeader_1x02_P2.54mm_Vertical, symbol Connector:Conn_01x02_Socket
- C7: footprint Capacitor_THT:C_Radial_D10.0mm_H12.5mm_P5.00mm -> Capacitor_THT:C_Radial_D5.0mm_H11.0mm_P2.00mm
- D15, D4, D5, D8: footprint Diode_SMD:D_MiniMELF -> Diode_THT:D_DO-35_SOD27_P7.62mm_Horizontal
Connections:
- net GND2: no longer D13.2 (A), D14.1 (K)
- net Live: no longer D11.2 (A), D12.1 (K)
- new net L_VFB: D11.2 (A), D12.1 (K), J6.1 (Pin_1)
- new net N_VFB: D13.2 (A), D14.1 (K), J6.2 (Pin_2)
Changed lines of the file:
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@@
 	)
 	(junction
-		(at 234.95 147.32)
+		(at 208.28 148.59)
 		(diameter 0)
 		(color 0 0 0 0)
 	)
 	(junction
-		(at 208.28 148.59)
+		(at 229.87 36.83)
 		(diameter 0)
 		(color 0 0 0 0)
 	)
 	(junction
-		(at 229.87 36.83)
+		(at 215.9 148.59)
 		(diameter 0)
 		(color 0 0 0 0)
 	)
 	(junction
-		(at 215.9 148.59)
+		(at 248.92 149.86)
+		(diameter 0)
+		(color 0 0 0 0)
+	)
+	(junction
+		(at 234.95 147.32)
 		(diameter 0)
 		(color 0 0 0 0)
@@
 	)
 	(junction
-		(at 248.92 149.86)
-		(diameter 0)
-		(color 0 0 0 0)
-	)
-	(junction
 		(at 172.72 162.56)
 		(diameter 0)
@@
 	(wire
 		(pts
-			(xy 234.95 147.32) (xy 265.43 147.32)
+			(xy 234.95 147.32) (xy 259.08 147.32)
 		)
 		(stroke
@@
 	(wire
 		(pts
-			(xy 248.92 149.86) (xy 265.43 149.86)
+			(xy 248.92 149.86) (xy 259.08 149.86)
 		)
 		(stroke
@@
 		)
 	)
-	(label "Live"
-		(at 257.81 147.32 0)
+	(label "L_VFB"
+		(at 251.46 147.32 0)
 		(effects
 			(font
@@
 		)
 	)
-	(label "Neutral"
-		(at 257.81 149.86 0)
+	(label "N_VFB"
+		(at 250.19 149.86 0)
 		(effects
 			(font
@@
 			)
 		)
-		(property "Footprint" "Diode_SMD:D_MiniMELF"
+		(property "Footprint" "Diode_THT:D_DO-35_SOD27_P7.62mm_Horizontal"
 			(at 29.845 179.07 0)
 			(hide yes)
@@
 	)
 	(symbol
+		(lib_id "Mechanical:MountingHole")
+		(at 43.18 104.14 0)
+		(unit 1)
+		(body_style 1)
+		(exclude_from_sim no)
+		(in_bom no)
+		(on_board yes)
+		(in_pos_files yes)
+		(dnp no)
+		(fields_autoplaced yes)
+		(property "Reference" "H4"
+			(at 45.72 104.1399 0)
+			(show_name no)
+			(do_not_autoplace no)
+			(effects
+				(font
+					(size 1.27 1.27)
+				)
+				(justify left)
+			)
+		)
+		(property "Value" "MountingHole"
+			(at 45.72 105.4099 0)
+			(hide yes)
+			(show_name no)
+			(do_not_autoplace no)
+			(effects
+				(font
+					(size 1.27 1.27)
+				)
+				(justify left)
+			)
+		)
+		(property "Footprint" "MountingHole:MountingHole_3.2mm_M3_Pad_Via"
+			(at 43.18 104.14 0)
+			(hide yes)
+			(show_name no)
+			(do_not_autoplace no)
+			(effects
+				(font
+					(size 1.27 1.27)
+				)
+			)
+		)
+		(property "Datasheet" ""
+			(at 43.18 104.14 0)
+			(hide yes)
+			(show_name no)
+			(do_not_autoplace no)
+			(effects
+				(font
+					(size 1.27 1.27)
+				)
+			)
+		)
+		(property "Description" "Mounting Hole without connection"
+			(at 43.18 104.14 0)
+			(hide yes)
+			(show_name no)
+			(do_not_autoplace no)
+			(effects
+				(font
+					(size 1.27 1.27)
+				)
+			)
+		)
+		(instances
+			(project "kicad"
+				(path "/40e0f264-5d7d-4080-96f9-03b6d8dad596"
+					(reference "H4")
+					(unit 1)
+				)
+			)
+		)
+	)
+	(symbol
 		(lib_id "Device:C_Small")
 		(at 63.5 58.42 90)
@@
 			)
 		)
-		(property "Footprint" "Diode_SMD:D_MiniMELF"
+		(property "Footprint" "Diode_THT:D_DO-35_SOD27_P7.62mm_Horizontal"
 			(at 65.405 182.88 0)
 			(hide yes)
@@
 			)
 		)
-		(property "Footprint" "Diode_SMD:D_MiniMELF"
+		(property "Footprint" "Diode_THT:D_DO-35_SOD27_P7.62mm_Horizontal"
 			(at 65.405 135.89 0)
 			(hide yes)
@@
 			)
 		)
-		(property "Footprint" "Diode_SMD:D_MiniMELF"
+		(property "Footprint" "Diode_THT:D_DO-35_SOD27_P7.62mm_Horizontal"
 			(at 203.835 154.94 0)
 			(hide yes)
@@
 			)
 		)
-		(property "Footprint" "Capacitor_THT:C_Radial_D10.0mm_H12.5mm_P5.00mm"
+		(property "Footprint" "Capacitor_THT:C_Radial_D5.0mm_H11.0mm_P2.00mm"
 			(at 227.33 148.59 0)
 			(hide yes)
@@
 					(unit 1)
 				)
+			)
+		)
+	)
+	(symbol
+		(lib_id "Connector:Conn_01x02_Socket")
+		(at 264.16 147.32 0)
+		(unit 1)
+		(body_style 1)
+		(exclude_from_sim no)
+		(in_bom yes)
+		(on_board yes)
+		(in_pos_files yes)
+		(dnp no)
+		(property "Reference" "J6"
+			(at 265.43 147.3199 0)
+			(show_name no)
+			(do_not_autoplace no)
+			(effects
+				(font
+					(size 1.27 1.27)
+				)
+				(justify left)
+			)
+		)
+		(property "Value" "Conn_01x02_Socket"
+			(at 258.064 153.162 0)
+			(hide yes)
+			(show_name no)
+			(do_not_autoplace no)
+			(effects
+				(font
+					(size 1.27 1.27)
+				)
+				(justify left)
+			)
+		)
+		(property "Footprint" "Connector_PinHeader_2.54mm:PinHeader_1x02_P2.54mm_Vertical"
+			(at 264.16 147.32 0)
+			(hide yes)
+			(show_name no)
+			(do_not_autoplace no)
+			(effects
+				(font
+					(size 1.27 1.27)
+				)
+			)
+		)
+		(property "Datasheet" ""
+			(at 264.16 147.32 0)
+			(hide yes)
+			(show_name no)
+			(do_not_autoplace no)
+			(effects
+				(font
+					(size 1.27 1.27)
+				)
+			)
+		)
+		(property "Description" "Generic connector, single row, 01x02, script generated"
+			(at 264.16 147.32 0)
+			(hide yes)
+			(show_name no)
+			(do_not_autoplace no)
+			(effects
+				(font
+					(size 1.27 1.27)
+				)
+			)
+		)
+		(pin "1"
+		)
+		(pin "2"
+		)
+		(instances
+			(project "kicad"
+				(path "/40e0f264-5d7d-4080-96f9-03b6d8dad596"
+					(reference "J6")
+					(unit 1)
+				)

Commit message: WORKING ON H Bridge kicad
Parts:
- added C12: 2.2uF, Capacitor_THT:C_Disc_D7.0mm_W2.5mm_P5.00mm, symbol Device:C_Small
- added C13: 100uF, Capacitor_THT:C_Disc_D7.0mm_W2.5mm_P5.00mm, symbol Device:C_Small
- added J10, J11, J12, J7, J8, J9: Conn_01x02_Socket, Connector_PinHeader_2.54mm:PinHeader_1x02_P2.54mm_Vertical, symbol Connector:Conn_01x02_Socket
- added R39, R41, R42: 33k, Resistor_THT:R_Axial_DIN0207_L6.3mm_D2.5mm_P7.62mm_Horizontal, symbol Device:R
- added R40: 10M, Resistor_THT:R_Axial_DIN0207_L6.3mm_D2.5mm_P7.62mm_Horizontal, symbol Device:R
- added RV6: 10k, Potentiometer_THT:Potentiometer_Bourns_3296W_Vertical, symbol Device:R_Potentiometer
- added U5: PC817, Package_DIP:DIP-4_W7.62mm, symbol Isolator:PC817
- C7: value 470uF 400V -> 10uF 400V
Connections:
- net 5V VREF: now also RV6.2, RV6.3
- net GND: now also C13.2, R40.1, U5.3; no longer C7.2, D15.2 (A), R15.1
- net INV: now also J11.1 (Pin_1), J12.1 (Pin_1); no longer D15.1 (K), R14.1, R15.2
- net at D12.2 (A), D14.2 (A): now also C7.2, C12.1, J8.2 (Pin_2)
- net at C7.1, D11.1 (K), D13.1 (K): now also C12.2, J7.1 (Pin_1); no longer R14.2
- new net: J7.2 (Pin_2), R39.1
- new net: R14.1, R39.2
- new net: J10.1 (Pin_1), R42.1
- new net: R41.1, R42.2
- new net: C13.1, J12.2 (Pin_2), R40.2, RV6.1, U5.4
- new net: R41.2, U5.1
- new net: D15.1 (K), J11.2 (Pin_2), R14.2, R15.2
- new net: D15.2 (A), J8.1 (Pin_1), R15.1
- new net: J9.2 (Pin_2), U5.2
Other:
- moved on the sheet: C1, C11, C2, C5, C6, C7, D11, D12, D13, D14, D15, D16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

Commit message: WORKING ON H Bridge kicad
Parts:
- removed C12: 2.2uF, Capacitor_THT:C_Disc_D7.0mm_W2.5mm_P5.00mm, symbol Device:C_Small
- removed C13: 100uF, Capacitor_THT:C_Disc_D7.0mm_W2.5mm_P5.00mm, symbol Device:C_Small
- removed C7: 10uF 400V, Capacitor_THT:C_Radial_D5.0mm_H11.0mm_P2.00mm, symbol Device:C_Polarized_Small
- removed D10, D11, D12, D13, D14, D7: 1N4007, Diode_THT:D_DO-41_SOD81_P10.16mm_Horizontal, symbol Diode:1N4007
- removed D15, D5, D8: BZV55B3V3, Diode_THT:D_DO-35_SOD27_P7.62mm_Horizontal, symbol Diode:BZV55B3V3
- removed D6, D9: LED, LED_THT:LED_D5.0mm, symbol Device:LED
- removed J10, J11, J12, J6, J7, J8, J9: Conn_01x02_Socket, Connector_PinHeader_2.54mm:PinHeader_1x02_P2.54mm_Vertical, symbol Connector:Conn_01x02_Socket
- removed R10, R14, R39, R41, R42, R6: 33k, Resistor_THT:R_Axial_DIN0207_L6.3mm_D2.5mm_P7.62mm_Horizontal, symbol Device:R
- removed R11, R15, R7: 10k, Resistor_THT:R_Axial_DIN0207_L6.3mm_D2.5mm_P7.62mm_Horizontal, symbol Device:R
- removed R12, R13, R5, R8: 1k, Resistor_THT:R_Axial_DIN0207_L6.3mm_D2.5mm_P7.62mm_Horizontal, symbol Device:R
- removed R19, R30: 390k, Resistor_THT:R_Axial_DIN0207_L6.3mm_D2.5mm_P7.62mm_Horizontal, symbol Device:R
- removed R4, R9: 4.7k, Resistor_THT:R_Axial_DIN0207_L6.3mm_D2.5mm_P7.62mm_Horizontal, symbol Device:R
- removed R40: 10M, Resistor_THT:R_Axial_DIN0207_L6.3mm_D2.5mm_P7.62mm_Horizontal, symbol Device:R
- removed RV3, RV4, RV6: 10k, Potentiometer_THT:Potentiometer_Bourns_3296W_Vertical, symbol Device:R_Potentiometer
- removed U3: LM358, Package_DIP:DIP-8_W7.62mm, symbol Amplifier_Operational:LM358
- removed U5: PC817, Package_DIP:DIP-4_W7.62mm, symbol Isolator:PC817
Other:
- added sheet isolated feedback (isolated feedback.kicad_sch)
- added sheet non isolated feedback (non isolated feedback.kicad_sch)
- added sheet protection circuit (protection circuit.kicad_sch)
- note removed: "HV ALARMS"
- note removed: "LV ALARMS"
- moved on the sheet: Q7, R36, R37

Commit message: WORKING ON H Bridge kicad
Parts:
- removed C1, C11, C2: 0.1uF 400V, Capacitor_THT:C_Rect_L13.5mm_W5.0mm_P10.00mm_FKS3_FKP3_MKS4, symbol Device:C
- removed C10: 1000uF 325V, Capacitor_THT:C_Radial_D10.0mm_H12.5mm_P5.00mm, symbol Device:C_Polarized_Small
- removed C3: 2.2uF, Capacitor_THT:C_Disc_D7.0mm_W2.5mm_P5.00mm, symbol Device:C_Small
- removed C4: 100nF, Capacitor_THT:C_Disc_D7.0mm_W2.5mm_P5.00mm, symbol Device:C_Small
- removed C5, C6: 330uF 16V, Capacitor_THT:C_Radial_D5.0mm_H11.0mm_P2.00mm, symbol Device:C_Polarized_Small
- removed C8: 1000uF 25V, Capacitor_THT:C_Radial_D10.0mm_H12.5mm_P5.00mm, symbol Device:C_Polarized_Small
- removed C9: 10uF 25V, Capacitor_THT:C_Radial_D5.0mm_H11.0mm_P2.00mm, symbol Device:C_Polarized_Small
- removed D1: LED, LED_THT:LED_D5.0mm, symbol Device:LED
- removed D16, D3: BA159, Diode_THT:D_DO-41_SOD81_P10.16mm_Horizontal, symbol Diode:BA159
- removed D4: BZV55B3V3, Diode_THT:D_DO-35_SOD27_P7.62mm_Horizontal, symbol Diode:BZV55B3V3
- removed J1, J5: Screw_Terminal_01x01, Connector_Wire:SolderWire-0.127sqmm_1x01_D0.48mm_OD1mm, symbol Connector:Screw_Terminal_01x01
- removed J2, J3, J4: Screw_Terminal_01x02, TerminalBlock_Phoenix:TerminalBlock_Phoenix_PT-1,5-2-5.0-H_1x02_P5.00mm_Horizontal, symbol Connector:Screw_Terminal_01x02
- removed Q1, Q2, Q5, Q6: IRF740, Package_TO_SOT_THT:TO-220-3_Vertical, symbol Transistor_FET:IRF740
- removed Q3, Q4: S8050, Package_TO_SOT_THT:TO-92_Inline, symbol Transistor_BJT:S8050
- removed Q7: BC547, Package_TO_SOT_THT:TO-92_Inline, symbol Transistor_BJT:BC547
- removed R1: 1k, Resistor_THT:R_Axial_DIN0207_L6.3mm_D2.5mm_P7.62mm_Horizontal, symbol Device:R
- removed R16, R23, R24, R26, R27, R28: 2.2k, Resistor_THT:R_Axial_DIN0207_L6.3mm_D2.5mm_P7.62mm_Horizontal, symbol Device:R
- removed R17, R20, R29, R31: 100, Resistor_THT:R_Axial_DIN0207_L6.3mm_D2.5mm_P7.62mm_Horizontal, symbol Device:R
- removed R18, R21, R32, R33, R36: 10k, Resistor_THT:R_Axial_DIN0207_L6.3mm_D2.5mm_P7.62mm_Horizontal, symbol Device:R
- removed R2: 51k, Resistor_THT:R_Axial_DIN0207_L6.3mm_D2.5mm_P7.62mm_Horizontal, symbol Device:R
- removed R22, R25, R3: 4.7k, Resistor_THT:R_Axial_DIN0207_L6.3mm_D2.5mm_P7.62mm_Horizontal, symbol Device:R
- removed R34: 370, Resistor_THT:R_Axial_DIN0207_L6.3mm_D2.5mm_P7.62mm_Horizontal, symbol Device:R
- removed R35: 20k, Resistor_THT:R_Axial_DIN0207_L6.3mm_D2.5mm_P7.62mm_Horizontal, symbol Device:R
- removed R37: 100k, Resistor_THT:R_Axial_DIN0207_L6.3mm_D2.5mm_P7.62mm_Horizontal, symbol Device:R
- removed R38: 47R, Resistor_THT:R_Axial_Power_L25.0mm_W6.4mm_P30.48mm, symbol Device:R
- removed RV2: 10k, Potentiometer_THT:Potentiometer_Bourns_3296W_Vertical, symbol Device:R_Potentiometer
- removed RV5: 150k, Potentiometer_THT:Potentiometer_Bourns_3296W_Vertical, symbol Device:R_Potentiometer
- removed U1: SG3525, Package_DIP:DIP-16_W7.62mm, symbol Regulator_Controller:SG3525
- removed U2, U4: PC817, Package_DIP:DIP-4_W7.62mm, symbol Isolator:PC817
Connections:
- no-connect marks 2 -> 0
Other:
- added sheet Full Bridge Bootstrap (Full Bridge Bootstrap.kicad_sch)
- added sheet SG3525 PWM (sg3525 pwm.kicad_sch)
- added sheet TL494 PMW (tl494 pwm.kicad_sch)
- note removed: "SNUBBER CIRCUIT"
- note removed: "Vout Ref"
- moved on the sheet: H1, H2, H3, H4
