File: SG3525 Solar Inverter/H Bridge/kicad/kicad.kicad_sch (KiCad schematic)
At the start: 4 parts

Commit message: WORKING ON H Bridge kicad
Other:
- added sheet DC DC Boost (dc dc boost.kicad_sch)
- moved on the sheet: H1, H2, H3, H4
Changed lines of the file:
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@@
 	(generator "eeschema")
 	(generator_version "10.0")
-	(paper "A3")
+	(paper "A4")
 	(title_block
 		(title "SG3525 Full Bridge Inverter")
@@
 	(symbol
 		(lib_id "Mechanical:MountingHole")
-		(at 199.39 73.66 0)
+		(at 190.5 116.84 0)
 		(unit 1)
 		(body_style 1)
@@
 		(fields_autoplaced yes)
 		(property "Reference" "H4"
-			(at 201.93 73.6599 0)
+			(at 193.04 116.8399 0)
 			(show_name no)
 			(do_not_autoplace no)
@@
 		)
 		(property "Value" "MountingHole"
-			(at 201.93 74.9299 0)
+			(at 193.04 118.1099 0)
 			(hide yes)
 			(show_name no)
@@
 		)
 		(property "Footprint" "MountingHole:MountingHole_3.2mm_M3_Pad_Via"
-			(at 199.39 73.66 0)
+			(at 190.5 116.84 0)
 			(hide yes)
 			(show_name no)
@@
 		)
 		(property "Datasheet" ""
-			(at 199.39 73.66 0)
+			(at 190.5 116.84 0)
 			(hide yes)
 			(show_name no)
@@
 		)
 		(property "Description" "Mounting Hole without connection"
-			(at 199.39 73.66 0)
+			(at 190.5 116.84 0)
 			(hide yes)
 			(show_name no)
@@
 	(symbol
 		(lib_id "Mechanical:MountingHole")
-		(at 199.39 68.58 0)
+		(at 190.5 111.76 0)
 		(unit 1)
 		(body_style 1)
@@
 		(fields_autoplaced yes)
 		(property "Reference" "H3"
-			(at 201.93 68.5799 0)
+			(at 193.04 111.7599 0)
 			(show_name no)
 			(do_not_autoplace no)
@@
 		)
 		(property "Value" "MountingHole"
-			(at 201.93 69.8499 0)
+			(at 193.04 113.0299 0)
 			(hide yes)
 			(show_name no)
@@
 		)
 		(property "Footprint" "MountingHole:MountingHole_3.2mm_M3_Pad_Via"
-			(at 199.39 68.58 0)
+			(at 190.5 111.76 0)
 			(hide yes)
 			(show_name no)
@@
 		)
 		(property "Datasheet" ""
-			(at 199.39 68.58 0)
+			(at 190.5 111.76 0)
 			(hide yes)
 			(show_name no)
@@
 		)
 		(property "Description" "Mounting Hole without connection"
-			(at 199.39 68.58 0)
+			(at 190.5 111.76 0)
 			(hide yes)
 			(show_name no)
@@
 	(symbol
 		(lib_id "Mechanical:MountingHole")
-		(at 199.39 58.42 0)
+		(at 190.5 101.6 0)
 		(unit 1)
 		(body_style 1)
@@
 		(fields_autoplaced yes)
 		(property "Reference" "H1"
-			(at 201.93 58.4199 0)
+			(at 193.04 101.5999 0)
 			(show_name no)
 			(do_not_autoplace no)
@@
 		)
 		(property "Value" "MountingHole"
-			(at 201.93 59.6899 0)
+			(at 193.04 102.8699 0)
 			(hide yes)
 			(show_name no)
@@
 		)
 		(property "Footprint" "MountingHole:MountingHole_3.2mm_M3_Pad_Via"
-			(at 199.39 58.42 0)
+			(at 190.5 101.6 0)
 			(hide yes)
 			(show_name no)
@@
 		)
 		(property "Datasheet" ""
-			(at 199.39 58.42 0)
+			(at 190.5 101.6 0)
 			(hide yes)
 			(show_name no)
@@
 		)
 		(property "Description" "Mounting Hole without connection"
-			(at 199.39 58.42 0)
+			(at 190.5 101.6 0)
 			(hide yes)
 			(show_name no)
@@
 	(symbol
 		(lib_id "Mechanical:MountingHole")
-		(at 199.39 63.5 0)
+		(at 190.5 106.68 0)
 		(unit 1)
 		(body_style 1)
@@
 		(fields_autoplaced yes)
 		(property "Reference" "H2"
-			(at 201.93 63.4999 0)
+			(at 193.04 106.6799 0)
 			(show_name no)
 			(do_not_autoplace no)
@@
 		)
 		(property "Value" "MountingHole"
-			(at 201.93 64.7699 0)
+			(at 193.04 107.9499 0)
 			(hide yes)
 			(show_name no)
@@
 		)
 		(property "Footprint" "MountingHole:MountingHole_3.2mm_M3_Pad_Via"
-			(at 199.39 63.5 0)
+			(at 190.5 106.68 0)
 			(hide yes)
 			(show_name no)
@@
 		)
 		(property "Datasheet" ""
-			(at 199.39 63.5 0)
+			(at 190.5 106.68 0)
 			(hide yes)
 			(show_name no)
@@
 		)
 		(property "Description" "Mounting Hole without connection"
-			(at 199.39 63.5 0)
+			(at 190.5 106.68 0)
 			(hide yes)
 			(show_name no)
@@
 	)
 	(sheet
-		(at 67.31 254)
+		(at 114.3 132.08)
 		(size 36.83 15.24)
 		(exclude_from_sim no)
@@
 		)
 		(property "Sheetname" "isolated feedback"
-			(at 67.31 253.2884 0)
+			(at 114.3 131.3684 0)
 			(show_name no)
 			(do_not_autoplace no)
@@
 		)
 		(property "Sheetfile" "isolated feedback.kicad_sch"
-			(at 67.31 269.8246 0)
+			(at 114.3 147.9046 0)
 			(show_name no)
 			(do_not_autoplace no)
@@
 	)
 	(sheet
-		(at 20.32 255.27)
-		(size 39.37 13.97)
+		(at 67.31 163.83)
+		(size 35.56 19.05)
 		(exclude_from_sim no)
 		(in_bom yes)
@@
 			(color 0 0 0 0)
 		)
-		(property "Sheetname" "protection circuit"
-			(at 20.32 254.5584 0)
+		(property "Sheetname" "DC DC Boost"
+			(at 67.31 163.1184 0)
 			(show_name no)
 			(do_not_autoplace no)
@@
 			)
 		)
-		(property "Sheetfile" "protection circuit.kicad_sch"
-			(at 20.32 269.8246 0)
+		(property "Sheetfile" "dc dc boost.kicad_sch"
+			(at 67.31 183.4646 0)
 			(show_name no)
 			(do_not_autoplace no)
@@
 			(project "kicad"
 				(path "/40e0f264-5d7d-4080-96f9-03b6d8dad596"
-					(page "3")
+					(page "8")
 				)
 			)
@@
 	)
 	(sheet
-		(at 67.31 231.14)
-		(size 36.83 15.24)
+		(at 67.31 133.35)
+		(size 35.56 13.97)
 		(exclude_from_sim no)
 		(in_bom yes)
@@
 			(color 0 0 0 0)
 		)
-		(property "Sheetname" "non isolated feedback"
-			(at 67.31 230.4284 0)
+		(property "Sheetname" "protection circuit"
+			(at 67.31 132.6384 0)
 			(show_name no)
 			(do_not_autoplace no)
@@
 			)
 		)
-		(property "Sheetfile" "non isolated feedback.kicad_sch"
-			(at 67.31 246.9646 0)
+		(property "Sheetfile" "protection circuit.kicad_sch"
+			(at 67.31 147.9046 0)
 			(show_name no)
 			(do_not_autoplace no)
@@
 			(project "kicad"
 				(path "/40e0f264-5d7d-4080-96f9-03b6d8dad596"
-					(page "4")
+					(page "3")
 				)
 			)
@@
 	)
 	(sheet
-		(at 19.05 199.39)
-		(size 39.37 17.78)
+		(at 114.3 109.22)
+		(size 36.83 15.24)
 		(exclude_from_sim no)
 		(in_bom yes)
@@
 			(color 0 0 0 0)
 		)
-		(property "Sheetname" "Full Bridge Bootstrap"
-			(at 19.05 198.6784 0)
+		(property "Sheetname" "non isolated feedback"
+			(at 114.3 108.5084 0)
 			(show_name no)
 			(do_not_autoplace no)
@@
 			)
 		)
-		(property "Sheetfile" "Full Bridge Bootstrap.kicad_sch"
-			(at 19.05 217.7546 0)
+		(property "Sheetfile" "non isolated feedback.kicad_sch"
+			(at 114.3 125.0446 0)
 			(show_name no)
 			(do_not_autoplace no)
@@
 			(project "kicad"
 				(path "/40e0f264-5d7d-4080-96f9-03b6d8dad596"
-					(page "6")
+					(page "4")
 				)
 			)
@@
 	)
 	(sheet
-		(at 20.32 227.33)
-		(size 35.56 17.78)
+		(at 66.04 77.47)
+		(size 36.83 17.78)
 		(exclude_from_sim no)
 		(in_bom yes)
@@
 			(color 0 0 0 0)
 		)
-		(property "Sheetname" "SG3525 PWM"
-			(at 20.32 226.6184 0)
+		(property "Sheetname" "Full Bridge Bootstrap"
+			(at 66.04 76.7584 0)
 			(show_name no)
 			(do_not_autoplace no)
@@
 			)
 		)
-		(property "Sheetfile" "sg3525 pwm.kicad_sch"
-			(at 20.32 245.6946 0)
+		(property "Sheetfile" "Full Bridge Bootstrap.kicad_sch"
+			(at 66.04 95.8346 0)
 			(show_name no)
 			(do_not_autoplace no)
@@
 			(project "kicad"
 				(path "/40e0f264-5d7d-4080-96f9-03b6d8dad596"
-					(page "2")
+					(page "6")
 				)
 			)
@@
 	)
 	(sheet
-		(at 66.04 199.39)
-		(size 38.1 17.78)
+		(at 67.31 109.22)
+		(size 35.56 15.24)
 		(exclude_from_sim no)
 		(in_bom yes)
@@
 			(color 0 0 0 0)
 		)
+		(property "Sheetname" "SG3525 PWM"
+			(at 67.31 108.5084 0)
+			(show_name no)
+			(do_not_autoplace no)
+			(effects
+				(font
+					(size 1.27 1.27)
+				)
+				(justify left bottom)
+			)
+		)
+		(property "Sheetfile" "sg3525 pwm.kicad_sch"
+			(at 67.31 125.0446 0)
+			(show_name no)
+			(do_not_autoplace no)
+			(effects
+				(font
+					(size 1.27 1.27)
+				)
+				(justify left top)
+			)
+		)
+		(instances
+			(project "kicad"
+				(path "/40e0f264-5d7d-4080-96f9-03b6d8dad596"
+					(page "2")
+				)
+			)
+		)
+	)
+	(sheet
+		(at 113.03 77.47)
+		(size 38.1 17.78)
+		(exclude_from_sim no)
+		(in_bom yes)
+		(on_board yes)
+		(dnp no)
+		(fields_autoplaced yes)
+		(stroke
+			(width 0.1524)
+			(type solid)
+		)
+		(fill
+			(color 0 0 0 0)
+		)
 		(property "Sheetname" "TL494 PMW"
-			(at 66.04 198.6784 0)
+			(at 113.03 76.7584 0)
 			(show_name no)
 			(do_not_autoplace no)
@@
 		)
 		(property "Sheetfile" "tl494 pwm.kicad_sch"
-			(at 66.04 217.7546 0)
-			(show_name no)
-			(do_not_autoplace no)
+			(at 113.03 95.8346 0)
+			(show_name no)
+			(do_not_autoplace no)
