File: SG3525 Solar Inverter/H Bridge/kicad/protection circuit.kicad_sch (KiCad schematic)
At the start: 21 parts, among them U3 LM358

Commit message: WORKING ON H Bridge kicad
Parts:
- added Q7: BC547, Package_TO_SOT_THT:TO-92_Inline, symbol Transistor_BJT:BC547
- added R36: 10k, Resistor_THT:R_Axial_DIN0207_L6.3mm_D2.5mm_P7.62mm_Horizontal, symbol Device:R
- added R37: 100k, Resistor_THT:R_Axial_DIN0207_L6.3mm_D2.5mm_P7.62mm_Horizontal, symbol Device:R
Connections:
- net GND: now also Q7.3 (E), R37.1
- net TR1: now also R36.2, R37.2
- new net: Q7.2 (B), R36.1
- new net SD: Q7.1 (C)
