File: SG3525 Solar Inverter/H Bridge/kicad/Full Bridge Bootstrap.kicad_sch (KiCad schematic)
At the start: 34 parts, among them J1 Screw_Terminal_01x01, J5 Screw_Terminal_01x01, Q1 IRF740, Q2 IRF740, Q3 S8050, Q4 S8050, Q5 IRF740, Q6 IRF740, U2 PC817, U4 PC817

Commit message: WORKING ON H Bridge kicad
Parts:
- added C14: 1000uF 325V, Capacitor_THT:C_Radial_D10.0mm_H12.5mm_P5.00mm, symbol Device:C_Polarized_Small
- added J13: Screw_Terminal_01x02, TerminalBlock_Phoenix:TerminalBlock_Phoenix_PT-1,5-2-5.0-H_1x02_P5.00mm_Horizontal, symbol Connector:Screw_Terminal_01x02
- added R47: 0.1R, Resistor_THT:R_Axial_DIN0207_L6.3mm_D2.5mm_P7.62mm_Horizontal, symbol Device:R
Connections:
- net +325V: now also C14.1, J13.1 (Pin_1)
- net GND: now also C14.2
- net GND2: now also J13.2 (Pin_2), R47.1; no longer Q2.3 (S), Q6.3 (S), R21.2, R33.2
- new net I Sense: Q2.3 (S), Q6.3 (S), R21.2, R33.2, R47.2
