File: SG3525 Solar Inverter/H Bridge/kicad/tl494 pwm.kicad_sch (KiCad schematic)
At the start: 17 parts, among them J13 Screw_Terminal_01x02, J14 Screw_Terminal_01x02, U7 TL494

Commit message: WORKING ON H Bridge kicad
Parts:
- removed C14: 1000uF 325V, Capacitor_THT:C_Radial_D10.0mm_H12.5mm_P5.00mm, symbol Device:C_Polarized_Small
- removed J13: Screw_Terminal_01x02, TerminalBlock_Phoenix:TerminalBlock_Phoenix_PT-1,5-2-5.0-H_1x02_P5.00mm_Horizontal, symbol Connector:Screw_Terminal_01x02
- removed R47: 370, Resistor_THT:R_Axial_DIN0207_L6.3mm_D2.5mm_P7.62mm_Horizontal, symbol Device:R
- added C20: 2.5uF 25V, Capacitor_THT:C_Radial_D5.0mm_H11.0mm_P2.00mm, symbol Device:C_Polarized_Small
- added R48: 10k, Resistor_THT:R_Axial_DIN0207_L6.3mm_D2.5mm_P7.62mm_Horizontal, symbol Device:R
- added RV9: 10k, Potentiometer_THT:Potentiometer_Bourns_3296W_Vertical, symbol Device:R_Potentiometer
- R43: value 4.7k -> 10k
Connections:
- net COMP is gone; now on net FB COMP: R45.2
- net INV is gone; now on net Vout Ref: C15.2, R45.1
- net 5V VREF: now also U7.14 (REF), C20.1, R48.2
- net CT: now also U7.5 (CT)
- net GND: now also RV8.1, U7.7 (GND), RV9.3; no longer RV8.3
- net OUTA: now also U7.9 (E1)
- net OUTB: now also U7.10 (E2)
- net RT: now also U7.6 (RT)
- net VC: now also U7.11 (C2), U7.12 (VCC), U7.8 (C1)
- net Vout Ref: now also U7.2 (1IN-)
- net VFB: now reaches U7.1 (1IN+)
- net FB COMP: now reaches U7.3 (FB)
- net DTC: now reaches U7.4 (DTC)
- net DTC: now also RV9.2
- net at R46.1: now also RV8.3; no longer RV8.1
- new net: C20.2, R48.1, RV9.1
Other:
- moved on the sheet: C15, C18, D2, J14, R44, R45, R46, RV8
