File: SG3525 Solar Inverter/H Bridge/kicad/_restore_backup_2026-10-04T13-43-24-165/kicad.kicad_pcb (KiCad board)
At the start: 2 copper layers, 106.7 x 65.5 mm, 76 parts, among them J2 Screw_Terminal_01x02, J3 Screw_Terminal_01x02, J4 Screw_Terminal_01x02, Q1 IRF740, Q2 IRF740, Q3 S8050, Q4 S8050, Q5 IRF740, Q6 IRF740, U1 SG3525, U2 PC817, U3 LM358, U4 PC817

Commit message: WORKING ON H Bridge kicad
Parts:
- removed C10: 1000uF 25V, Capacitor_THT:C_Radial_D10.0mm_H12.5mm_P5.00mm
- removed J2, J3, J4: Screw_Terminal_01x02, TerminalBlock_Phoenix:TerminalBlock_Phoenix_PT-1,5-2-5.0-H_1x02_P5.00mm_Horizontal
- added D2: BYV79-100, Package_TO_SOT_THT:TO-220-2_Vertical, F.Cu at (-104.4, 130.5)
- added J1: Conn_01x02_Pin, Connector_PinHeader_1.00mm:PinHeader_1x02_P1.00mm_Vertical, F.Cu at (-135.8, 92.1)
- added R19: 0, Resistor_THT:R_Axial_DIN0207_L6.3mm_D2.5mm_P7.62mm_Horizontal, F.Cu at (-106.5, 109.1)
- added RV1: 10k, Potentiometer_THT:Potentiometer_Bourns_3296W_Vertical, F.Cu at (-124.8, 109.7)
- C7, C8: footprint Capacitor_THT:C_Radial_D10.0mm_H12.5mm_P5.00mm -> Capacitor_THT:C_Radial_D16.0mm_H25.0mm_P7.50mm
- moved R30 242.5 mm to (-88.2, 118.1), turned to 0 degrees
- moved R3 238.6 mm to (-130.5, 98.3), turned to 0 degrees
- moved R1 236.7 mm to (-135.7, 98.3)
- moved D4 233.4 mm to (-118.1, 114.9), turned to 0 degrees
- moved D1 226.8 mm to (-134.5, 110.9), turned to -90 degrees
- moved RV2 226.5 mm to (-113.2, 99.6), turned to 0 degrees
- moved C8 189.7 mm to (-88.9, 146.0), turned to 0 degrees
- moved R14 8.75 mm to (187.5, 126.8), turned to 0 degrees
- moved R15 8.51 mm to (195.2, 131.2), turned to 180 degrees
- moved C3 5.81 mm to (109.9, 138.6), turned to 90 degrees
- moved D15 3.71 mm to (183.7, 129.5)
- moved C7 3.51 mm to (181.1, 113.9), turned to 0 degrees
- moved R2 2.93 mm to (109.9, 129.4)
- moved D11 2.27 mm to (179.9, 102.2)
- moved D12 2.27 mm to (190.3, 86.8)
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Connections:
- C5 pad 2: /Live -> Net-(C5-Pad2)
- C6 pad 2: /Neutral -> Net-(C6-Pad2)
Other:
- board size 106.7 x 65.5 mm -> 92.9 x 65.5 mm
