File: SG3525 Solar Inverter/H Bridge/kicad/_restore_backup_2026-10-04T13-43-24-165/kicad.kicad_sch (KiCad schematic)
At the start: 75 parts, among them J2 Screw_Terminal_01x02, J3 Screw_Terminal_01x02, J4 Screw_Terminal_01x02, Q1 IRF740, Q2 IRF740, Q3 S8050, Q4 S8050, Q5 IRF740, Q6 IRF740, U1 SG3525, U2 PC817, U3 LM358, U4 PC817

Commit message: WORKING ON H Bridge kicad
Parts:
- removed C10: 1000uF 25V, Capacitor_THT:C_Radial_D10.0mm_H12.5mm_P5.00mm, symbol Device:C_Polarized_Small
- removed J2, J3, J4: Screw_Terminal_01x02, TerminalBlock_Phoenix:TerminalBlock_Phoenix_PT-1,5-2-5.0-H_1x02_P5.00mm_Horizontal, symbol Connector:Screw_Terminal_01x02
- added J1: Conn_01x02_Pin, Connector_PinHeader_1.00mm:PinHeader_1x02_P1.00mm_Vertical, symbol Connector:Conn_01x02_Pin
- added R19, R30: 0, Resistor_THT:R_Axial_DIN0207_L6.3mm_D2.5mm_P7.62mm_Horizontal, symbol Device:R
- C7, C8: footprint Capacitor_THT:C_Radial_D10.0mm_H12.5mm_P5.00mm -> Capacitor_THT:C_Radial_D16.0mm_H25.0mm_P7.50mm
Connections:
- net +12V: now also J1.1 (Pin_1)
- net GND: now also J1.2 (Pin_2)
- net Live: now also R19.2; no longer C5.2
- net Neutral: now also R30.2; no longer C6.2
- new net: C5.2, R19.1
- new net: C6.2, R30.1
